Commit message: modif du lidar

File: workspaceRos/src/robot_description/urdf/robot.urdf.xacro (robot description, xacro)
@@ -102,5 +102,5 @@
    <joint name="hokuyo_joint" type="fixed">
       <axis xyz="0 1 0" />
-      <origin xyz="0 0 0.2" rpy="0 0 0"/>
+      <origin xyz="0 0 0.25" rpy="0 0 0"/>
       <parent link="chassis"/>
       <child link="hokuyo_link"/>
@@ -109,5 +109,5 @@
    <link name="hokuyo_link">
       <collision>
-         <origin xyz="0 0 0" rpy="0 0 0"/>
+         <origin xyz="0 0 -0.01" rpy="0 0 0"/>
          <geometry>
     	    <cylinder radius="0.05" length="0.2"/>
@@ -115,5 +115,5 @@
       </collision>
       <visual>
-         <origin xyz="0 0 0" rpy="0 0 0"/>
+         <origin xyz="0 0 -0.01" rpy="0 0 0"/>
          <geometry>
             <cylinder radius="0.05" length="0.2"/>
@@ -129,5 +129,5 @@
    <gazebo reference="hokuyo_link">
       <sensor type="ray" name="head_hokuyo_sensor">
-         <pose>0 0 0.5 0 0 0</pose>
+         <pose>0 0 0.0 0 0 0</pose>
          <visualize>true</visualize>
          <update_rate>2</update_rate>
@@ -280,6 +280,6 @@
          <!-- ENTER BASE LINK NAME -->
          <robotBaseFrame>base_link</robotBaseFrame>
-         <publishWheelTF>false</publishWheelTF>
-         <publishTf>true</publishTf>
+         <publishWheelTF>true</publishWheelTF>
+         <publishTf>false</publishTf>
          <publishWheelJointState>true</publishWheelJointState>
          <legacyMode>false</legacyMode>

Commit message: "ajout du bras au robot"

File: workspaceRos/src/robot_description/urdf/robot.urdf.xacro (robot description, xacro)
@@ -2,4 +2,5 @@
 <robot name="monRobot" xmlns:xacro="http://ros.org/wiki/xacro">
   <xacro:include filename="$(find robot_description)/urdf/robot.wheels.xacro"/>
+  <xacro:include filename="$(find robot_description)/urdf/arm.xacro"/>
   <xacro:macro name="default_inertial" params="mass">
     <inertial>
@@ -8,5 +9,5 @@
     </inertial>
   </xacro:macro>
-  <link name="base_link"/> <!-- permet d'utiliser Move Base -->
+  <link name="base_link"/> <!-- permet d'utiliser Move Base   <xacro:property name="arm_position" value="0.17"/>-->
   <joint name="base_joint" type="fixed">
     <parent link="base_link"/>
@@ -47,4 +48,5 @@
     <parent link="chassis"/>
   </joint>
+  <!-- Wheels -->
   <link name="left_wheel">
     <collision>
@@ -77,4 +79,5 @@
     <xacro:default_inertial mass="0.3"/>
   </link>
+  <!-- Wheel's Joints -->
   <joint type="continuous" name="left_wheel_hinge">
     <origin xyz="0.1 0.13 0.1" rpy="0 0 0"/>
@@ -89,4 +92,12 @@
     <axis xyz="0 1 0"/>
   </joint>
+  <!-- Arm Joint -->
+  <joint name="chassis_arm_joint" type="fixed">
+    <axis xyz="0 0 1"/>
+    <origin rpy="0 0 0" xyz="${arm_position} 0 0.2"/>
+    <parent link="chassis"/>
+    <child link="arm_1_link"/>
+  </joint>
+  <!-- Hokuyo Joint -->
   <joint name="hokuyo_joint" type="fixed">
     <axis xyz="0 1 0" />

Commit message: modif lidar

File: workspaceRos/src/robot_description/urdf/robot.urdf.xacro (robot description, xacro)
@@ -102,5 +102,5 @@
    <joint name="hokuyo_joint" type="fixed">
       <axis xyz="0 1 0" />
-      <origin xyz="0 0 0.25" rpy="0 0 0"/>
+      <origin xyz="0 0 0.22" rpy="0 0 0"/>
       <parent link="chassis"/>
       <child link="hokuyo_link"/>
@@ -109,5 +109,5 @@
    <link name="hokuyo_link">
       <collision>
-         <origin xyz="0 0 -0.01" rpy="0 0 0"/>
+         <origin xyz="0 0 -0.03" rpy="0 0 0"/>
          <geometry>
     	    <cylinder radius="0.05" length="0.2"/>
@@ -115,5 +115,5 @@
       </collision>
       <visual>
-         <origin xyz="0 0 -0.01" rpy="0 0 0"/>
+         <origin xyz="0 0 -0.03" rpy="0 0 0"/>
          <geometry>
             <cylinder radius="0.05" length="0.2"/>
@@ -129,5 +129,5 @@
    <gazebo reference="hokuyo_link">
       <sensor type="ray" name="head_hokuyo_sensor">
-         <pose>0 0 0.0 0 0 0</pose>
+         <pose>0 0 0.5 0 0 0</pose>
          <visualize>true</visualize>
          <update_rate>2</update_rate>
@@ -164,5 +164,5 @@
    <!-- joint Chassis-Camera -->
    <joint name="camera_joint" type="fixed">
-      <origin xyz="0.22 0 0.1" rpy="0 0.3 0"/>
+      <origin xyz="0.22 0 0.09" rpy="0 0.3 0"/>
       <parent link="chassis"/>
       <child link="camera_link"/>
@@ -280,6 +280,6 @@
          <!-- ENTER BASE LINK NAME -->
          <robotBaseFrame>base_link</robotBaseFrame>
-         <publishWheelTF>true</publishWheelTF>
-         <publishTf>false</publishTf>
+         <publishWheelTF>false</publishWheelTF>
+         <publishTf>true</publishTf>
          <publishWheelJointState>true</publishWheelJointState>
          <legacyMode>false</legacyMode>

Commit message: solve conflict robot.urdf.xacro

File: workspaceRos/src/robot_description/urdf/robot.urdf.xacro (robot description, xacro)
@@ -16,39 +16,4 @@
       <origin xyz="0 0 0.01" rpy="0 0 0"/>
    </joint>
-<<<<<<< HEAD
-  <link name="chassis">
-    <collision>
-      <origin xyz="0 0 .1" rpy="0 0 0"/>
-      <geometry>
-        <box size="0.4 0.2 0.1"/>
-      </geometry>
-    </collision>
-    <visual>
-      <origin xyz="0 0 .1" rpy="0 0 0"/>
-      <geometry>
-        <box size="0.4 0.2 0.1"/>
-      </geometry>
-    </visual>
-    <xacro:default_inertial mass="2.0"/>
-  </link>
-  <link name="caster">
-    <collision>
-      <geometry>
-        <sphere radius="0.05"/>
-      </geometry>
-    </collision>
-    <visual>
-      <geometry>
-        <sphere radius="0.05"/>
-      </geometry>
-    </visual>
-    <xacro:default_inertial mass="0.01"/>
-  </link>
-  <joint name="caster_to_chassis" type="fixed">
-    <origin xyz="-0.15 0 0.05" rpy="0 0 0"/>
-    <child link="caster"/>
-    <parent link="chassis"/>
-  </joint>
-=======
    <!-- Chassis-->
    <link name="chassis">
@@ -67,5 +32,4 @@
      <xacro:default_inertial mass="2.0"/>
    </link>
->>>>>>> 06c67a4350b1a4dbc1f57f1e9bc8ccef10583e76
    <!-- Roue Libre-->
    <link name="caster">

Commit message: solve conflict robot.urdf.xacro 2

File: workspaceRos/src/robot_description/urdf/robot.urdf.xacro (robot description, xacro)
@@ -105,35 +105,4 @@
     <child link="arm_1_link"/>
   </joint>
-<<<<<<< HEAD
-    <inertial>
-      <mass value="1e-5" />
-      <origin xyz="0 0 0" rpy="0 0 0"/>
-      <inertia ixx="1e-6" ixy="0" ixz="0" iyy="1e-6" iyz="0" izz="1e-6" />
-    </inertial>
-  </link>
-  <!-- hokuyo -->
-  <gazebo reference="hokuyo_link">
-    <sensor type="ray" name="head_hokuyo_sensor">
-      <pose>0 0 0 0 0 0</pose>
-      <visualize>true</visualize>
-      <update_rate>2</update_rate>
-      <ray>
-        <scan>
-          <horizontal>
-            <samples>30</samples>
-            <resolution>1</resolution>
-            <min_angle>-3.1415</min_angle>
-            <max_angle>3.1415</max_angle>
-          </horizontal>
-        </scan>
-        <range>
-          <min>0.10</min>
-          <max>30.0</max>
-          <resolution>0.01</resolution>
-        </range>
-        <noise>
-          <type>gaussian</type>
-          <!-- Noise parameters based on published spec for Hokuyo laser
-=======
    <!-- Joint Chassis-Lidar-->
    <joint name="hokuyo_joint" type="fixed">
@@ -186,5 +155,4 @@
                <type>gaussian</type>
                <!-- Noise parameters based on published spec for Hokuyo laser
->>>>>>> 06c67a4350b1a4dbc1f57f1e9bc8ccef10583e76
                achieving "+-30mm" accuracy at range < 10m.  A mean of 0.0m and
                stddev of 0.01m will put 99.7% of samples within 0.03m of the true

Commit message: replace camera

File: workspaceRos/src/robot_description/urdf/robot.urdf.xacro (robot description, xacro)
@@ -1,4 +1,5 @@
 <?xml version="1.0"?>
 <robot name="monRobot" xmlns:xacro="http://ros.org/wiki/xacro">
+  <xacro:property name="length_4" value="0.1" /> <!-- laser arm -->
   <xacro:include filename="$(find robot_description)/urdf/robot.wheels.xacro"/>
   <xacro:include filename="$(find robot_description)/urdf/arm.xacro"/>
@@ -105,13 +106,13 @@
     <child link="arm_1_link"/>
   </joint>
-   <!-- Joint Chassis-Lidar-->
-   <joint name="hokuyo_joint" type="fixed">
+  <!-- Joint Chassis-Lidar-->
+  <!-- <joint name="hokuyo_joint" type="fixed">
       <axis xyz="0 1 0" />
       <origin xyz="0 0 0.22" rpy="0 0 0"/>
       <parent link="chassis"/>
       <child link="hokuyo_link"/>
-   </joint>
+   </joint>-->
    <!-- Hokuyo Laser -->
-   <link name="hokuyo_link">
+ <!--  <link name="hokuyo_link">
       <collision>
          <origin xyz="0 0 -0.03" rpy="0 0 0"/>
@@ -131,7 +132,7 @@
          <inertia ixx="1e-6" ixy="0" ixz="0" iyy="1e-6" iyz="0" izz="1e-6" />
       </inertial>
-   </link>
+   </link>-->
    <!-- Plugin Hokuyo -->
-   <gazebo reference="hokuyo_link">
+  <!-- <gazebo reference="hokuyo_link">
       <sensor type="ray" name="head_hokuyo_sensor">
          <pose>0 0 0.5 0 0 0</pose>
@@ -153,10 +154,10 @@
             </range>
             <noise>
-               <type>gaussian</type>
+               <type>gaussian</type>-->
                <!-- Noise parameters based on published spec for Hokuyo laser
                achieving "+-30mm" accuracy at range < 10m.  A mean of 0.0m and
                stddev of 0.01m will put 99.7% of samples within 0.03m of the true
                reading. -->
-               <mean>0.0</mean>
+           <!--     <mean>0.0</mean>
                <stddev>0.01</stddev>
             </noise>
@@ -167,13 +168,13 @@
          </plugin>
       </sensor>
-   </gazebo>
-   <!-- joint Chassis-Camera -->
-   <joint name="camera_joint" type="fixed">
-      <origin xyz="0.22 0 0.09" rpy="0 0.3 0"/>
-      <parent link="chassis"/>
-      <child link="camera_link"/>
+   </gazebo>-->
+   <!-- joint Bras-Camera -->
+   <joint name="cameraBras_joint" type="fixed">
+      <origin xyz="0 0 ${length_4}" rpy="0 0 0"/>
+      <parent link="laser"/>
+      <child link="cameraBras_link"/>
    </joint>
    <!-- Camera -->
-   <link name="camera_link">
+   <link name="cameraBras_link">
       <collision>
          <origin xyz="0 0 0" rpy="0 0 0"/>
@@ -195,7 +196,7 @@
       </inertial>
    </link>
-   <xacro:property name="camera_link" value="0.4" /> <!-- Size of square 'camera' box -->
+   <xacro:property name="camera_link" value="0.1" /> <!-- Size of square 'camera' box -->
    <!-- Plugin Camera -->
-   <gazebo reference="camera_link">
+   <gazebo reference="cameraBras_link">
       <sensor type="camera" name="camera1">
          <update_rate>30.0</update_rate>

Commit message: suprime doublon ds robot.urdf.xacro

File: workspaceRos/src/robot_description/urdf/robot.urdf.xacro (robot description, xacro)
@@ -221,5 +221,5 @@
       </inertial>
    </link>
-   <xacro:property name="camera_link" value="0.4" /> <!-- Size of square 'camera' box -->
+   <xacro:property name="camera_link" value="0.4" /> <!--size of 'camera' box-->
    <!-- Plugin Camera -->
    <gazebo reference="camera_link">
@@ -304,29 +304,3 @@
       </plugin>
    </gazebo>
-  <!-- Controllers -->
-   <gazebo>
-      <plugin name="wheels_controller" filename="libgazebo_ros_diff_drive.so">
-         <commandTopic>cmd_vel</commandTopic>
-         <odometryTopic>odom</odometryTopic>
-         <odometryFrame>odom</odometryFrame>
-         <odometrySource>world</odometrySource>
-         <publishOdomTF>true</publishOdomTF>
-         <!-- ENTER BASE LINK NAME -->
-         <robotBaseFrame>base_link</robotBaseFrame>
-         <publishWheelTF>false</publishWheelTF>
-         <publishTf>true</publishTf>
-         <publishWheelJointState>true</publishWheelJointState>
-         <legacyMode>false</legacyMode>
-         <updateRate>30</updateRate>
-         <!-- ENTER LEFT JOINT NAME -->
-         <leftJoint>left_wheel_hinge</leftJoint>
-         <!-- ENTER RIGHT JOINT NAME -->
-         <rightJoint>right_wheel_hinge</rightJoint>
-         <wheelSeparation>0.31</wheelSeparation>
-         <wheelDiameter>0.1</wheelDiameter>
-         <wheelAcceleration>0.1</wheelAcceleration>
-         <wheelTorque>10</wheelTorque>
-         <rosDebugLevel>na</rosDebugLevel>
-      </plugin>
-   </gazebo>
 </robot>

Commit message: add camera

File: workspaceRos/src/robot_description/urdf/robot.urdf.xacro (robot description, xacro)
@@ -134,5 +134,5 @@
    </link>-->
    <!-- Plugin Hokuyo -->
-  <!-- <gazebo reference="hokuyo_link">
+  <!--  <gazebo reference="hokuyo_link">
       <sensor type="ray" name="head_hokuyo_sensor">
          <pose>0 0 0.5 0 0 0</pose>
@@ -159,5 +159,5 @@
                stddev of 0.01m will put 99.7% of samples within 0.03m of the true
                reading. -->
-           <!--     <mean>0.0</mean>
+            <!--    <mean>0.0</mean>
                <stddev>0.01</stddev>
             </noise>
@@ -168,5 +168,73 @@
          </plugin>
       </sensor>
-   </gazebo>-->
+   </gazebo> -->
+    <!-- joint Chassis-Camera -->
+   <joint name="camera_joint" type="fixed">
+      <origin xyz="0.22 0 0.09" rpy="0 0.3 0"/>
+      <parent link="chassis"/>
+      <child link="camera_link"/>
+   </joint>
+   <!-- Camera -->
+   <link name="camera_link">
+      <collision>
+         <origin xyz="0 0 0" rpy="0 0 0"/>
+         <geometry>
+            <box size="0.04 0.04 0.04"/>
+         </geometry>
+      </collision>
+      <visual>
+         <origin xyz="0 0 0" rpy="0 0 0"/>
+         <geometry>
+            <box size="0.04 0.04 0.04"/>
+         </geometry>
+         <material name="red"/>
+      </visual>
+      <inertial>
+         <mass value="1e-5" />
+         <origin xyz="0 0 0" rpy="0 0 0"/>
+         <inertia ixx="1e-6" ixy="0" ixz="0" iyy="1e-6" iyz="0" izz="1e-6" />
+      </inertial>
+   </link>
+   <xacro:property name="camera_link" value="0.4" /> <!-- Size of square 'camera' box -->
+   <!-- Plugin Camera -->
+   <gazebo reference="camera_link">
+      <sensor type="camera" name="camera1">
+         <update_rate>30.0</update_rate>
+         <camera name="head">
+            <horizontal_fov>1.3962634</horizontal_fov>
+            <image>
+               <width>800</width>
+               <height>800</height>
+               <format>R8G8B8</format>
+            </image>
+            <clip>
+               <near>0.02</near>
+               <far>300</far>
+            </clip>
+            <noise>
+               <type>gaussian</type>
+               <!-- Noise is sampled independently per pixel on each frame.
+               That pixel's noise value is added to each of its color
+               channels, which at that point lie in the range [0,1]. -->
+               <mean>0.0</mean>
+               <stddev>0.007</stddev>
+            </noise>
+         </camera>
+         <plugin name="camera_controller" filename="libgazebo_ros_camera.so">
+            <alwaysOn>true</alwaysOn>
+            <updateRate>0.0</updateRate>
+            <cameraName>rrbot/camera1</cameraName>
+            <imageTopicName>image_raw</imageTopicName>
+            <cameraInfoTopicName>camera_info</cameraInfoTopicName>
+            <frameName>camera_link</frameName>
+            <hackBaseline>0.07</hackBaseline>
+            <distortionK1>0.0</distortionK1>
+            <distortionK2>0.0</distortionK2>
+            <distortionK3>0.0</distortionK3>
+            <distortionT1>0.0</distortionT1>
+            <distortionT2>0.0</distortionT2>
+         </plugin>
+      </sensor>
+   </gazebo>
    <!-- joint Bras-Camera -->
    <joint name="cameraBras_joint" type="fixed">

Commit message: upgdate support lidar

File: workspaceRos/src/robot_description/urdf/robot.urdf.xacro (robot description, xacro)
@@ -132,17 +132,44 @@
     <child link="arm_1_link"/>
   </joint>
-  <!-- Joint Chassis-Hokuyo-->
-  <!-- <joint name="hokuyo_joint" type="fixed">
+   <!-- Joint Chassis-Support Hokuyo-->
+   <!--<joint name="support_hokuyo_joint" type="fixed">
       <axis xyz="0 1 0" />
       <origin xyz="0 0 0.22" rpy="0 0 0"/>
       <parent link="chassis"/>
+      <child link="hokuyo_support"/>
+   </joint>-->
+   <!-- Hokuyo Support -->
+   <!--<link name="hokuyo_support">
+      <collision>
+         <origin xyz="0 0 -0.03" rpy="0 0 0"/>
+         <geometry>
+    	    <cylinder radius="0.05" length="0.14"/>
+         </geometry>
+      </collision>
+      <visual>
+         <origin xyz="0 0 -0.03" rpy="0 0 0"/>
+         <geometry>
+            <cylinder radius="0.05" length="0.14"/>
+         </geometry>
+      </visual>
+      <inertial>
+         <mass value="1e-5" />
+         <origin xyz="0 0 0" rpy="0 0 0"/>
+         <inertia ixx="1e-6" ixy="0" ixz="0" iyy="1e-6" iyz="0" izz="1e-6" />
+      </inertial>
+   </link>-->
+   <!-- Joint Support-Hokuyo-->
+   <!--<joint name="hokuyo_joint" type="fixed">
+      <axis xyz="0 1 0" />
+      <origin xyz="0 0 0.06" rpy="0 0 0"/>
+      <parent link="hokuyo_support"/>
       <child link="hokuyo_link"/>
    </joint>-->
    <!-- Hokuyo Laser -->
- <!--  <link name="hokuyo_link">
+   <!-- <link name="hokuyo_link">
       <collision>
          <origin xyz="0 0 -0.03" rpy="0 0 0"/>
          <geometry>
-    	    <cylinder radius="0.05" length="0.2"/>
+    	    <cylinder radius="0.05" length="0.05"/>
          </geometry>
       </collision>
@@ -150,5 +177,5 @@
          <origin xyz="0 0 -0.03" rpy="0 0 0"/>
          <geometry>
-            <cylinder radius="0.05" length="0.2"/>
+            <cylinder radius="0.05" length="0.05"/>
          </geometry>
       </visual>
@@ -201,5 +228,5 @@
       <child link="camera_link"/>
    </joint>
-   <!-- Camera -->
+   <!-- Chassis-Camera -->
    <link name="camera_link">
       <collision>
@@ -223,5 +250,5 @@
    </link>
    <xacro:property name="camera_link" value="0.4" /> <!--size of 'camera' box-->
-   <!-- Plugin Camera -->
+   <!-- Plugin Chassis-Camera -->
    <gazebo reference="camera_link">
       <sensor type="camera" name="camera1">
@@ -269,5 +296,5 @@
       <child link="cameraBras_link"/>
    </joint>
-   <!-- Camera -->
+   <!-- Bras-Camera -->
    <link name="cameraBras_link">
       <collision>
@@ -291,5 +318,5 @@
    </link>
    <xacro:property name="camera_link" value="0.1" /> <!-- Size of square 'camera' box -->
-   <!-- Plugin Camera -->
+   <!-- Plugin Bras-Camera -->
    <gazebo reference="cameraBras_link">
       <sensor type="camera" name="camera1">
