Commit message: change camera name

File: workspaceRos/src/robot_description/urdf/robot.urdf.xacro (robot description, xacro)
@@ -1,4 +1,5 @@
 <?xml version="1.0"?>
 <robot name="monRobot" xmlns:xacro="http://ros.org/wiki/xacro">
+  <xacro:property name="length_4" value="0.1" /> <!-- laser arm -->
   <xacro:include filename="$(find robot_description)/urdf/robot.wheels.xacro"/>
   <xacro:include filename="$(find robot_description)/urdf/arm.xacro"/>
@@ -131,13 +132,13 @@
     <child link="arm_1_link"/>
   </joint>
-   <!-- Joint Chassis-Hokuyo-->
-   <joint name="hokuyo_joint" type="fixed">
+  <!-- Joint Chassis-Hokuyo-->
+  <!-- <joint name="hokuyo_joint" type="fixed">
       <axis xyz="0 1 0" />
       <origin xyz="0 0 0.22" rpy="0 0 0"/>
       <parent link="chassis"/>
       <child link="hokuyo_link"/>
-   </joint>
+   </joint>-->
    <!-- Hokuyo Laser -->
-   <link name="hokuyo_link">
+ <!--  <link name="hokuyo_link">
       <collision>
          <origin xyz="0 0 -0.03" rpy="0 0 0"/>
@@ -157,7 +158,7 @@
          <inertia ixx="1e-6" ixy="0" ixz="0" iyy="1e-6" iyz="0" izz="1e-6" />
       </inertial>
-   </link>
+   </link>-->
    <!-- Plugin Hokuyo -->
-   <gazebo reference="hokuyo_link">
+  <!--  <gazebo reference="hokuyo_link">
       <sensor type="ray" name="head_hokuyo_sensor">
          <pose>0 0 0.5 0 0 0</pose>
@@ -179,10 +180,10 @@
             </range>
             <noise>
-               <type>gaussian</type>
+               <type>gaussian</type>-->
                <!-- Noise parameters based on published spec for Hokuyo laser
                achieving "+-30mm" accuracy at range < 10m.  A mean of 0.0m and
                stddev of 0.01m will put 99.7% of samples within 0.03m of the true
                reading. -->
-               <mean>0.0</mean>
+            <!--    <mean>0.0</mean>
                <stddev>0.01</stddev>
             </noise>
@@ -193,6 +194,6 @@
          </plugin>
       </sensor>
-   </gazebo>
-   <!-- joint Chassis-Camera -->
+   </gazebo> -->
+    <!-- joint Chassis-Camera -->
    <joint name="camera_joint" type="fixed">
       <origin xyz="0.22 0 0.09" rpy="0 0.3 0"/>
@@ -221,5 +222,5 @@
       </inertial>
    </link>
-   <xacro:property name="camera_link" value="0.4" /> <!-- Size of square 'camera' box -->
+   <xacro:property name="camera_link" value="0.4" /> <!--size of 'camera' box-->
    <!-- Plugin Camera -->
    <gazebo reference="camera_link">
@@ -262,4 +263,72 @@
       </sensor>
    </gazebo>
+   <!-- joint Bras-Camera -->
+   <joint name="cameraBras_joint" type="fixed">
+      <origin xyz="0 0 ${length_4}" rpy="0 0 0"/>
+      <parent link="laser"/>
+      <child link="cameraBras_link"/>
+   </joint>
+   <!-- Camera -->
+   <link name="cameraBras_link">
+      <collision>
+         <origin xyz="0 0 0" rpy="0 0 0"/>
+         <geometry>
+            <box size="0.04 0.04 0.04"/>
+         </geometry>
+      </collision>
+      <visual>
+         <origin xyz="0 0 0" rpy="0 0 0"/>
+         <geometry>
+            <box size="0.04 0.04 0.04"/>
+         </geometry>
+         <material name="red"/>
+      </visual>
+      <inertial>
+         <mass value="1e-5" />
+         <origin xyz="0 0 0" rpy="0 0 0"/>
+         <inertia ixx="1e-6" ixy="0" ixz="0" iyy="1e-6" iyz="0" izz="1e-6" />
+      </inertial>
+   </link>
+   <xacro:property name="camera_link" value="0.1" /> <!-- Size of square 'camera' box -->
+   <!-- Plugin Camera -->
+   <gazebo reference="cameraBras_link">
+      <sensor type="camera" name="camera1">
+         <update_rate>30.0</update_rate>
+         <camera name="head">
+            <horizontal_fov>1.3962634</horizontal_fov>
+            <image>
+               <width>800</width>
+               <height>800</height>
+               <format>R8G8B8</format>
+            </image>
+            <clip>
+               <near>0.02</near>
+               <far>300</far>
+            </clip>
+            <noise>
+               <type>gaussian</type>
+               <!-- Noise is sampled independently per pixel on each frame.
+               That pixel's noise value is added to each of its color
+               channels, which at that point lie in the range [0,1]. -->
+               <mean>0.0</mean>
+               <stddev>0.007</stddev>
+            </noise>
+         </camera>
+         <plugin name="camera_controller" filename="libgazebo_ros_camera.so">
+            <alwaysOn>true</alwaysOn>
+            <updateRate>0.0</updateRate>
+            <cameraName>rrbot/cameraBras</cameraName>
+            <imageTopicName>image_raw</imageTopicName>
+            <cameraInfoTopicName>camera_info</cameraInfoTopicName>
+            <frameName>camera_link</frameName>
+            <hackBaseline>0.07</hackBaseline>
+            <distortionK1>0.0</distortionK1>
+            <distortionK2>0.0</distortionK2>
+            <distortionK3>0.0</distortionK3>
+            <distortionT1>0.0</distortionT1>
+            <distortionT2>0.0</distortionT2>
+         </plugin>
+      </sensor>
+   </gazebo>
    <!-- Joint Chassis-GPS-->
    <joint name="gps_joint" type="fixed">
@@ -304,29 +373,3 @@
       </plugin>
    </gazebo>
-  <!-- Controllers -->
-   <gazebo>
-      <plugin name="wheels_controller" filename="libgazebo_ros_diff_drive.so">
-         <commandTopic>cmd_vel</commandTopic>
-         <odometryTopic>odom</odometryTopic>
-         <odometryFrame>odom</odometryFrame>
-         <odometrySource>world</odometrySource>
-         <publishOdomTF>true</publishOdomTF>
-         <!-- ENTER BASE LINK NAME -->
-         <robotBaseFrame>base_link</robotBaseFrame>
-         <publishWheelTF>false</publishWheelTF>
-         <publishTf>true</publishTf>
-         <publishWheelJointState>true</publishWheelJointState>
-         <legacyMode>false</legacyMode>
-         <updateRate>30</updateRate>
-         <!-- ENTER LEFT JOINT NAME -->
-         <leftJoint>left_wheel_hinge</leftJoint>
-         <!-- ENTER RIGHT JOINT NAME -->
-         <rightJoint>right_wheel_hinge</rightJoint>
-         <wheelSeparation>0.31</wheelSeparation>
-         <wheelDiameter>0.1</wheelDiameter>
-         <wheelAcceleration>0.1</wheelAcceleration>
-         <wheelTorque>10</wheelTorque>
-         <rosDebugLevel>na</rosDebugLevel>
-      </plugin>
-   </gazebo>
 </robot>

Commit message: debut sonar

File: workspaceRos/src/robot_description/urdf/robot.urdf.xacro (robot description, xacro)
@@ -400,3 +400,30 @@
       </plugin>
    </gazebo>
+   <!-- Joint Chassis-Sonar-->
+   <!--<joint name="sonar_joint" type="fixed">
+      <axis xyz="0 0 0" />
+      <origin xyz="0.2 0.05 0.09" rpy="0 0 0"/>
+      <parent link="chassis"/>
+      <child link="sonar_link"/>
+   </joint>-->
+   <!-- Sonar -->
+   <!--<link name="sonar_link">
+      <collision>
+         <origin xyz="0 0 0" rpy="1.5707 1.5707 1.5707"/>
+         <geometry>
+    	    <cylinder radius="0.02" length="0.015"/>
+         </geometry>
+      </collision>
+      <visual>
+         <origin xyz="0 0 0" rpy="1.5707 1.5707 1.5707"/>
+         <geometry>
+            <cylinder radius="0.02" length="0.015"/>
+         </geometry>
+      </visual>
+      <inertial>
+         <mass value="1e-5" />
+         <origin xyz="0 0 0" rpy="0 0 0"/>
+         <inertia ixx="1e-6" ixy="0" ixz="0" iyy="1e-6" iyz="0" izz="1e-6" />
+      </inertial>
+   </link>-->
 </robot>

Commit message: modification du xacro

File: workspaceRos/src/robot_description/urdf/robot.urdf.xacro (robot description, xacro)
@@ -358,72 +358,4 @@
       </sensor>
    </gazebo>
-   <!-- joint Bras-Camera -->
-   <joint name="cameraBras_joint" type="fixed">
-      <origin xyz="0 0 ${length_4}" rpy="0 0 0"/>
-      <parent link="laser"/>
-      <child link="cameraBras_link"/>
-   </joint>
-   <!-- Bras-Camera -->
-   <link name="cameraBras_link">
-      <collision>
-         <origin xyz="0 0 0" rpy="0 0 0"/>
-         <geometry>
-            <box size="0.04 0.04 0.04"/>
-         </geometry>
-      </collision>
-      <visual>
-         <origin xyz="0 0 0" rpy="0 0 0"/>
-         <geometry>
-            <box size="0.04 0.04 0.04"/>
-         </geometry>
-         <material name="red"/>
-      </visual>
-      <inertial>
-         <mass value="1e-5" />
-         <origin xyz="0 0 0" rpy="0 0 0"/>
-         <inertia ixx="1e-6" ixy="0" ixz="0" iyy="1e-6" iyz="0" izz="1e-6" />
-      </inertial>
-   </link>
-   <xacro:property name="camera_link" value="0.1" /> <!-- Size of square 'camera' box -->
-   <!-- Plugin Bras-Camera -->
-   <gazebo reference="cameraBras_link">
-      <sensor type="camera" name="camera1">
-         <update_rate>30.0</update_rate>
-         <camera name="head">
-            <horizontal_fov>1.3962634</horizontal_fov>
-            <image>
-               <width>800</width>
-               <height>800</height>
-               <format>R8G8B8</format>
-            </image>
-            <clip>
-               <near>0.02</near>
-               <far>300</far>
-            </clip>
-            <noise>
-               <type>gaussian</type>
-               <!-- Noise is sampled independently per pixel on each frame.
-               That pixel's noise value is added to each of its color
-               channels, which at that point lie in the range [0,1]. -->
-               <mean>0.0</mean>
-               <stddev>0.007</stddev>
-            </noise>
-         </camera>
-         <plugin name="camera_controller" filename="libgazebo_ros_camera.so">
-            <alwaysOn>true</alwaysOn>
-            <updateRate>0.0</updateRate>
-            <cameraName>rrbot/camera1</cameraName>
-            <imageTopicName>image_raw</imageTopicName>
-            <cameraInfoTopicName>camera_info</cameraInfoTopicName>
-            <frameName>camera_link</frameName>
-            <hackBaseline>0.07</hackBaseline>
-            <distortionK1>0.0</distortionK1>
-            <distortionK2>0.0</distortionK2>
-            <distortionK3>0.0</distortionK3>
-            <distortionT1>0.0</distortionT1>
-            <distortionT2>0.0</distortionT2>
-         </plugin>
-      </sensor>
-   </gazebo>
    <!-- Joint Chassis-GPS-->
    <joint name="gps_joint" type="fixed">

Commit message: On a regler les problemes d urdf

File: workspaceRos/src/robot_description/urdf/robot.urdf.xacro (robot description, xacro)
@@ -1,5 +1,4 @@
 <?xml version="1.0"?>
 <robot name="monRobot" xmlns:xacro="http://ros.org/wiki/xacro">
-  <xacro:property name="length_4" value="0.1" /> <!-- laser arm -->
   <xacro:include filename="$(find robot_description)/urdf/robot.wheels.xacro"/>
   <xacro:include filename="$(find robot_description)/urdf/arm.xacro"/>
@@ -31,5 +30,5 @@
          </geometry>
       </visual>
-     <xacro:default_inertial mass="10.0"/>
+     <xacro:default_inertial mass="2.0"/>
    </link>
    <!-- Roue Libre-->
@@ -92,5 +91,5 @@
       <axis xyz="0 1 0"/>
    </joint>
-   <!-- Joint Chassis-Roue Gauche-->
+   <!-- Joint Chassis-Roue Right-->
    <joint type="continuous" name="right_wheel_hinge">
       <origin xyz="0.1 -0.13 0.1" rpy="0 0 0"/>
@@ -132,17 +131,17 @@
     <child link="arm_1_link"/>
   </joint>
-   <!-- Joint Chassis-Support Hokuyo-->
-   <!--<joint name="support_hokuyo_joint" type="fixed">
+   <!-- Joint Chassis-Hokuyo-->
+   <joint name="hokuyo_joint" type="fixed">
       <axis xyz="0 1 0" />
       <origin xyz="0 0 0.22" rpy="0 0 0"/>
       <parent link="chassis"/>
-      <child link="hokuyo_support"/>
-   </joint>-->
-   <!-- Hokuyo Support -->
-   <!--<link name="hokuyo_support">
+      <child link="hokuyo_link"/>
+   </joint>
+   <!-- Hokuyo Laser -->
+   <link name="hokuyo_link">
       <collision>
          <origin xyz="0 0 -0.03" rpy="0 0 0"/>
          <geometry>
-    	    <cylinder radius="0.05" length="0.14"/>
+    	    <cylinder radius="0.05" length="0.2"/>
          </geometry>
       </collision>
@@ -150,5 +149,5 @@
          <origin xyz="0 0 -0.03" rpy="0 0 0"/>
          <geometry>
-            <cylinder radius="0.05" length="0.14"/>
+            <cylinder radius="0.05" length="0.2"/>
          </geometry>
       </visual>
@@ -158,34 +157,7 @@
          <inertia ixx="1e-6" ixy="0" ixz="0" iyy="1e-6" iyz="0" izz="1e-6" />
       </inertial>
-   </link>-->
-   <!-- Joint Support-Hokuyo-->
-   <!--<joint name="hokuyo_joint" type="fixed">
-      <axis xyz="0 1 0" />
-      <origin xyz="0 0 0.06" rpy="0 0 0"/>
-      <parent link="hokuyo_support"/>
-      <child link="hokuyo_link"/>
-   </joint>-->
-   <!-- Hokuyo Laser -->
-   <!-- <link name="hokuyo_link">
-      <collision>
-         <origin xyz="0 0 -0.03" rpy="0 0 0"/>
-         <geometry>
-    	    <cylinder radius="0.05" length="0.05"/>
-         </geometry>
-      </collision>
-      <visual>
-         <origin xyz="0 0 -0.03" rpy="0 0 0"/>
-         <geometry>
-            <cylinder radius="0.05" length="0.05"/>
-         </geometry>
-      </visual>
-      <inertial>
-         <mass value="1e-5" />
-         <origin xyz="0 0 0" rpy="0 0 0"/>
-         <inertia ixx="1e-6" ixy="0" ixz="0" iyy="1e-6" iyz="0" izz="1e-6" />
-      </inertial>
-   </link>-->
+   </link>
    <!-- Plugin Hokuyo -->
-  <!--  <gazebo reference="hokuyo_link">
+   <gazebo reference="hokuyo_link">
       <sensor type="ray" name="head_hokuyo_sensor">
          <pose>0 0 0.5 0 0 0</pose>
@@ -207,10 +179,10 @@
             </range>
             <noise>
-               <type>gaussian</type>-->
+               <type>gaussian</type>
                <!-- Noise parameters based on published spec for Hokuyo laser
                achieving "+-30mm" accuracy at range < 10m.  A mean of 0.0m and
                stddev of 0.01m will put 99.7% of samples within 0.03m of the true
                reading. -->
-            <!--    <mean>0.0</mean>
+               <mean>0.0</mean>
                <stddev>0.01</stddev>
             </noise>
@@ -221,6 +193,6 @@
          </plugin>
       </sensor>
-   </gazebo> -->
-    <!-- joint Chassis-Camera -->
+   </gazebo>
+   <!-- joint Chassis-Camera -->
    <joint name="camera_joint" type="fixed">
       <origin xyz="0.22 0 0.09" rpy="0 0.3 0"/>
@@ -290,5 +262,9 @@
       </sensor>
    </gazebo>
-   <!-- joint Bras-Camera -->
+   <!-- Plugin Chassis-Camera -->
+   <!-- Plugin Chassis-Camera -->
+   <!-- Plugin Chassis-Camera -->
+   <!-- Plugin Chassis-Camera -->
+<!-- joint Bras-Camera -->
    <joint name="cameraBras_joint" type="fixed">
       <origin xyz="0 0 ${length_4}" rpy="0 0 0"/>
@@ -317,8 +293,8 @@
       </inertial>
    </link>
-   <xacro:property name="camera_link" value="0.1" /> <!-- Size of square 'camera' box -->
+   <xacro:property name="cameraBras_link" value="0.1" /> <!-- Size of square 'camera' box -->
    <!-- Plugin Camera -->
    <gazebo reference="cameraBras_link">
-      <sensor type="camera" name="camera1">
+      <sensor type="camera" name="cameraBras">
          <update_rate>30.0</update_rate>
          <camera name="head">
@@ -400,30 +376,3 @@
       </plugin>
    </gazebo>
-   <!-- Joint Chassis-Sonar-->
-   <!--<joint name="sonar_joint" type="fixed">
-      <axis xyz="0 0 0" />
-      <origin xyz="0.2 0.05 0.09" rpy="0 0 0"/>
-      <parent link="chassis"/>
-      <child link="sonar_link"/>
-   </joint>-->
-   <!-- Sonar -->
-   <!--<link name="sonar_link">
-      <collision>
-         <origin xyz="0 0 0" rpy="1.5707 1.5707 1.5707"/>
-         <geometry>
-    	    <cylinder radius="0.02" length="0.015"/>
-         </geometry>
-      </collision>
-      <visual>
-         <origin xyz="0 0 0" rpy="1.5707 1.5707 1.5707"/>
-         <geometry>
-            <cylinder radius="0.02" length="0.015"/>
-         </geometry>
-      </visual>
-      <inertial>
-         <mass value="1e-5" />
-         <origin xyz="0 0 0" rpy="0 0 0"/>
-         <inertia ixx="1e-6" ixy="0" ixz="0" iyy="1e-6" iyz="0" izz="1e-6" />
-      </inertial>
-   </link>-->
 </robot>

Commit message: merge des codes

File: workspaceRos/src/robot_description/urdf/robot.urdf.xacro (robot description, xacro)
@@ -268,5 +268,5 @@
 <!-- joint Bras-Camera -->
    <joint name="cameraBras_joint" type="fixed">
-      <origin xyz="0 0 ${length_4}" rpy="0 0 0"/>
+      <origin xyz="0 0 ${length_4}" rpy="0 -1.7 0"/>
       <parent link="laser"/>
       <child link="cameraBras_link"/>

Commit message: support hokuyo ajouter

File: workspaceRos/src/robot_description/urdf/robot.urdf.xacro (robot description, xacro)
@@ -131,9 +131,36 @@
     <child link="arm_1_link"/>
   </joint>
+   <!-- Joint Chassis-Support Hokuyo-->
+   <joint name="support_hokuyo_joint" type="fixed">
+      <axis xyz="0 1 0" />
+      <origin xyz="0 0 0.22" rpy="0 0 0"/>
+      <parent link="chassis"/>
+      <child link="hokuyo_support"/>
+   </joint>
+   <!-- Hokuyo Support -->
+   <link name="hokuyo_support">
+      <collision>
+         <origin xyz="0 0 -0.03" rpy="0 0 0"/>
+         <geometry>
+    	    <cylinder radius="0.05" length="0.14"/>
+         </geometry>
+      </collision>
+      <visual>
+         <origin xyz="0 0 -0.03" rpy="0 0 0"/>
+         <geometry>
+            <cylinder radius="0.05" length="0.14"/>
+         </geometry>
+      </visual>
+      <inertial>
+         <mass value="1e-5" />
+         <origin xyz="0 0 0" rpy="0 0 0"/>
+         <inertia ixx="1e-6" ixy="0" ixz="0" iyy="1e-6" iyz="0" izz="1e-6" />
+      </inertial>
+   </link>
    <!-- Joint Chassis-Hokuyo-->
    <joint name="hokuyo_joint" type="fixed">
       <axis xyz="0 1 0" />
       <origin xyz="0 0 0.22" rpy="0 0 0"/>
-      <parent link="chassis"/>
+      <parent link="hokuyo_support"/>
       <child link="hokuyo_link"/>
    </joint>
@@ -143,5 +170,5 @@
          <origin xyz="0 0 -0.03" rpy="0 0 0"/>
          <geometry>
-    	    <cylinder radius="0.05" length="0.2"/>
+    	    <cylinder radius="0.05" length="0.05"/>
          </geometry>
       </collision>
@@ -149,5 +176,5 @@
          <origin xyz="0 0 -0.03" rpy="0 0 0"/>
          <geometry>
-            <cylinder radius="0.05" length="0.2"/>
+            <cylinder radius="0.05" length="0.05"/>
          </geometry>
       </visual>
@@ -162,5 +189,5 @@
       <sensor type="ray" name="head_hokuyo_sensor">
          <pose>0 0 0.5 0 0 0</pose>
-         <visualize>true</visualize>
+         <visualize>false</visualize>
          <update_rate>2</update_rate>
          <ray>
@@ -376,3 +403,30 @@
       </plugin>
    </gazebo>
+   <!-- Joint Chassis-Sonar-->
+   <!--<joint name="sonar_joint" type="fixed">
+      <axis xyz="0 0 0" />
+      <origin xyz="0.2 0.05 0.09" rpy="0 0 0"/>
+      <parent link="chassis"/>
+      <child link="sonar_link"/>
+   </joint>-->
+   <!-- Sonar -->
+   <!--<link name="sonar_link">
+      <collision>
+         <origin xyz="0 0 0" rpy="1.5707 1.5707 1.5707"/>
+         <geometry>
+    	    <cylinder radius="0.02" length="0.015"/>
+         </geometry>
+      </collision>
+      <visual>
+         <origin xyz="0 0 0" rpy="1.5707 1.5707 1.5707"/>
+         <geometry>
+            <cylinder radius="0.02" length="0.015"/>
+         </geometry>
+      </visual>
+      <inertial>
+         <mass value="1e-5" />
+         <origin xyz="0 0 0" rpy="0 0 0"/>
+         <inertia ixx="1e-6" ixy="0" ixz="0" iyy="1e-6" iyz="0" izz="1e-6" />
+      </inertial>
+   </link>-->
 </robot>

Commit message: debut de transition vers pthon2 ; findcontorut non regle

File: workspaceRos/src/robot_description/urdf/robot.urdf.xacro (robot description, xacro)
@@ -10,10 +10,10 @@
   </xacro:macro>
    <!-- Robot -->
-   <link name="base_link"/> <!-- permet d'utiliser Move Base -->
+   <!--link name="base_link"/> <permet d'utiliser Move Base >
    <joint name="base_joint" type="fixed">
       <parent link="base_link"/>
       <child link="chassis" />
       <origin xyz="0 0 0.01" rpy="0 0 0"/>
-   </joint>
+   </joint-->
    <!-- Chassis-->
    <link name="chassis">

Commit message: correction du probleme de tf

File: workspaceRos/src/robot_description/urdf/robot.urdf.xacro (robot description, xacro)
@@ -10,10 +10,10 @@
   </xacro:macro>
    <!-- Robot -->
-   <!--link name="base_link"/> <permet d'utiliser Move Base >
+   <link name="base_link"/> <!--permet d'utiliser Move Base -->
    <joint name="base_joint" type="fixed">
       <parent link="base_link"/>
       <child link="chassis" />
       <origin xyz="0 0 0.01" rpy="0 0 0"/>
-   </joint-->
+   </joint>
    <!-- Chassis-->
    <link name="chassis">
