Commit message: update gps et camera

File: workspaceRos/src/robot_description/urdf/robot.urdf (robot description, URDF)
Before this commit: robot monRobot, 7 links, 6 joints
Links:
- added link gps_link, mass 1e-5; collision cylinder length=0.03 radius=0.03; visual cylinder length=0.03 radius=0.03
- link camera_link: geometry collision box size=0.04 0.04 0.04; visual box size=0.04 0.04 0.04
- link hokuyo_link: geometry collision cylinder length=0.2 radius=0.05; visual cylinder length=0.2 radius=0.05
Joints:
- added joint gps_joint: type fixed, parent chassis, child gps_link, origin xyz=-0.15 0 0.17 rpy=0 0 0, axis 0 0 0
- joint camera_joint: origin xyz=0.1 0 0.2 rpy=0 0 0 -> xyz=0.22 0 0.1 rpy=0 0.3 0

File: workspaceRos/src/robot_description/urdf/robot.urdf.xacro (robot description, xacro)
@@ -1,247 +1,298 @@
 <?xml version="1.0"?>
 <robot name="monRobot" xmlns:xacro="http://ros.org/wiki/xacro">
-  <xacro:include filename="$(find robot_description)/urdf/robot.wheels.xacro"/>
-  <xacro:macro name="default_inertial" params="mass">
-    <inertial>
-      <mass value="${mass}" />
-      <inertia ixx="0.01" ixy="0.0" ixz="0.0" iyy="0.01" iyz="0.0" izz="0.01" />
-    </inertial>
-  </xacro:macro>
-  <link name="base_link"/> <!-- permet d'utiliser Move Base -->
-  <joint name="base_joint" type="fixed">
-    <parent link="base_link"/>
-    <child link="chassis" />
-    <origin xyz="0 0 0.01" rpy="0 0 0"/>
-  </joint>
-  <link name="chassis">
-    <collision>
-      <origin xyz="0 0 .1" rpy="0 0 0"/>
-      <geometry>
-        <box size="0.4 0.2 0.1"/>
-      </geometry>
-    </collision>
-    <visual>
-      <origin xyz="0 0 .1" rpy="0 0 0"/>
-      <geometry>
-        <box size="0.4 0.2 0.1"/>
-      </geometry>
-    </visual>
-    <xacro:default_inertial mass="2.0"/>
-  </link>
-  <link name="caster">
-    <collision>
-      <geometry>
-        <sphere radius="0.05"/>
-      </geometry>
-    </collision>
-    <visual>
-      <geometry>
-        <sphere radius="0.05"/>
-      </geometry>
-    </visual>
-    <xacro:default_inertial mass="0.01"/>
-  </link>
-  <joint name="caster_to_chassis" type="fixed">
-    <origin xyz="-0.15 0 0.05" rpy="0 0 0"/>
-    <child link="caster"/>
-    <parent link="chassis"/>
-  </joint>
-  <link name="left_wheel">
-    <collision>
-      <origin xyz="0 0 0" rpy="0 1.5707 1.5707"/>
-      <geometry>
-        <cylinder radius="0.1" length="0.05"/>
-      </geometry>
-    </collision>
-    <visual>
-      <origin xyz="0 0 0" rpy="0 1.5707 1.5707"/>
-      <geometry>
-        <cylinder radius="0.1" length="0.05"/>
-      </geometry>
-    </visual>
-    <xacro:default_inertial mass="0.3"/>
-  </link>
-  <link name="right_wheel">
-    <collision>
-      <origin xyz="0 0 0" rpy="0 1.5707 1.5707"/>
-      <geometry>
-        <cylinder radius="0.1" length="0.05"/>
-      </geometry>
-    </collision>
-    <visual>
-      <origin xyz="0 0 0" rpy="0 1.5707 1.5707"/>
-      <geometry>
-        <cylinder radius="0.1" length="0.05"/>
-      </geometry>
-    </visual>
-    <xacro:default_inertial mass="0.3"/>
-  </link>
-  <joint type="continuous" name="left_wheel_hinge">
-    <origin xyz="0.1 0.13 0.1" rpy="0 0 0"/>
-    <child link="left_wheel"/>
-    <parent link="chassis"/>
-    <axis xyz="0 1 0"/>
-  </joint>
-  <joint type="continuous" name="right_wheel_hinge">
-    <origin xyz="0.1 -0.13 0.1" rpy="0 0 0"/>
-    <child link="right_wheel"/>
-    <parent link="chassis"/>
-    <axis xyz="0 1 0"/>
-  </joint>
-  <joint name="hokuyo_joint" type="fixed">
-    <axis xyz="0 1 0" />
-    <origin xyz="0 0 0.2" rpy="0 0 0"/>
-    <parent link="chassis"/>
-    <child link="hokuyo_link"/>
-  </joint>
-  <!-- Hokuyo Laser -->
-  <link name="hokuyo_link">
-    <collision>
-      <origin xyz="0 0 0" rpy="0 0 0"/>
-      <geometry>
-    	<box size="0.1 0.1 0.1"/>
-      </geometry>
-    </collision>
-    <visual>
-      <origin xyz="0 0 0" rpy="0 0 0"/>
-      <geometry>
-        <sphere radius="0.1"/>
-      </geometry>
-    </visual>
-    <inertial>
-      <mass value="1e-5" />
-      <origin xyz="0 0 0" rpy="0 0 0"/>
-      <inertia ixx="1e-6" ixy="0" ixz="0" iyy="1e-6" iyz="0" izz="1e-6" />
-    </inertial>
-  </link>
-  <!-- hokuyo -->
-  <gazebo reference="hokuyo_link">
-    <sensor type="ray" name="head_hokuyo_sensor">
-      <pose>0 0 0 0 0 0</pose>
-      <visualize>true</visualize>
-      <update_rate>2</update_rate>
-      <ray>
-        <scan>
-          <horizontal>
-            <samples>720</samples>
-            <resolution>1</resolution>
-            <min_angle>-3.1415</min_angle>
-            <max_angle>3.1415</max_angle>
-          </horizontal>
-        </scan>
-        <range>
-          <min>0.10</min>
-          <max>30.0</max>
-          <resolution>0.01</resolution>
-        </range>
-        <noise>
-          <type>gaussian</type>
-          <!-- Noise parameters based on published spec for Hokuyo laser
+   <xacro:include filename="$(find robot_description)/urdf/robot.wheels.xacro"/>
+   <xacro:macro name="default_inertial" params="mass">
+      <inertial>
+         <mass value="${mass}" />
+         <inertia ixx="0.01" ixy="0.0" ixz="0.0"
+                  iyy="0.01" iyz="0.0"
+                  izz="0.01" />
+       </inertial>
+   </xacro:macro>
+<!-- Robot -->
+   <link name="base_link"/> <!-- permet d'utiliser Move Base -->
+   <joint name="base_joint" type="fixed">
+      <parent link="base_link"/>
+      <child link="chassis" />
+      <origin xyz="0 0 0.01" rpy="0 0 0"/>
+   </joint>
+   <!-- Chassis-->
+   <link name="chassis">
+      <collision>
+         <origin xyz="0 0 .1" rpy="0 0 0"/>
+         <geometry>
+            <box size="0.4 0.2 0.1"/>
+         </geometry>
+      </collision>
+      <visual>
+         <origin xyz="0 0 .1" rpy="0 0 0"/>
+         <geometry>
+            <box size="0.4 0.2 0.1"/>
+         </geometry>
+      </visual>
+     <xacro:default_inertial mass="2.0"/>
+   </link>
+   <!-- Roue Libre-->
+   <link name="caster">
+      <collision>
+         <geometry>
+            <sphere radius="0.05"/>
+         </geometry>
+      </collision>
+      <visual>
+         <geometry>
+           <sphere radius="0.05"/>
+         </geometry>
+      </visual>
+      <xacro:default_inertial mass="0.01"/>
+   </link>
+   <!-- Joint Chassis-Roue Libre-->
+   <joint name="caster_to_chassis" type="fixed">
+      <origin xyz="-0.15 0 0.05" rpy="0 0 0"/>
+      <child link="caster"/>
+      <parent link="chassis"/>
+   </joint>
+   <!-- Roue Gauche-->
+   <link name="left_wheel">
+      <collision>
+         <origin xyz="0 0 0" rpy="0 1.5707 1.5707"/>
+         <geometry>
+            <cylinder radius="0.1" length="0.05"/>
+         </geometry>
+      </collision>
+      <visual>
+         <origin xyz="0 0 0" rpy="0 1.5707 1.5707"/>
+         <geometry>
+              <cylinder radius="0.1" length="0.05"/>
+         </geometry>
+      </visual>
+      <xacro:default_inertial mass="0.3"/>
+   </link>
+   <!-- Roue Droite-->
+   <link name="right_wheel">
+      <collision>
+         <origin xyz="0 0 0" rpy="0 1.5707 1.5707"/>
+         <geometry>
+            <cylinder radius="0.1" length="0.05"/>
+         </geometry>
+      </collision>
+      <visual>
+         <origin xyz="0 0 0" rpy="0 1.5707 1.5707"/>
+         <geometry>
+            <cylinder radius="0.1" length="0.05"/>
+         </geometry>
+      </visual>
+      <xacro:default_inertial mass="0.3"/>
+   </link>
+   <!-- Joint Chassis-Roue Gauche-->
+   <joint type="continuous" name="left_wheel_hinge">
+      <origin xyz="0.1 0.13 0.1" rpy="0 0 0"/>
+      <child link="left_wheel"/>
+      <parent link="chassis"/>
+      <axis xyz="0 1 0"/>
+   </joint>
+   <!-- Joint Chassis-Roue Gauche-->
+   <joint type="continuous" name="right_wheel_hinge">
+      <origin xyz="0.1 -0.13 0.1" rpy="0 0 0"/>
+      <child link="right_wheel"/>
+      <parent link="chassis"/>
+      <axis xyz="0 1 0"/>
+   </joint>
+   <!-- Joint Chassis-Laser-->
+   <joint name="hokuyo_joint" type="fixed">
+      <axis xyz="0 1 0" />
+      <origin xyz="0 0 0.2" rpy="0 0 0"/>
+      <parent link="chassis"/>
+      <child link="hokuyo_link"/>
+   </joint>
+   <!-- Hokuyo Laser -->
+   <link name="hokuyo_link">
+      <collision>
+         <origin xyz="0 0 0" rpy="0 0 0"/>
+         <geometry>
+    	    <cylinder radius="0.05" length="0.2"/>
+         </geometry>
+      </collision>
+      <visual>
+         <origin xyz="0 0 0" rpy="0 0 0"/>
+         <geometry>
+            <cylinder radius="0.05" length="0.2"/>
+         </geometry>
+      </visual>
+      <inertial>
+         <mass value="1e-5" />
+         <origin xyz="0 0 0" rpy="0 0 0"/>
+         <inertia ixx="1e-6" ixy="0" ixz="0" iyy="1e-6" iyz="0" izz="1e-6" />
+      </inertial>
+   </link>
+   <!-- Plugin Hokuyo -->
+   <gazebo reference="hokuyo_link">
+      <sensor type="ray" name="head_hokuyo_sensor">
+         <pose>0 0 0.5 0 0 0</pose>
+         <visualize>true</visualize>
+         <update_rate>2</update_rate>
+         <ray>
+            <scan>
+               <horizontal>
+                  <samples>50</samples>
+                  <resolution>1</resolution>
+                  <min_angle>-3.1415</min_angle>
+                  <max_angle>3.1415</max_angle>
+               </horizontal>
+            </scan>
+            <range>
+               <min>0.10</min>
+               <max>30.0</max>
+               <resolution>0.01</resolution>
+            </range>
+            <noise>
+               <type>gaussian</type>
+               <!-- Noise parameters based on published spec for Hokuyo laser
                achieving "+-30mm" accuracy at range < 10m.  A mean of 0.0m and
                stddev of 0.01m will put 99.7% of samples within 0.03m of the true
                reading. -->
-          <mean>0.0</mean>
-          <stddev>0.01</stddev>
-        </noise>
-      </ray>
-      <plugin name="gazebo_ros_head_hokuyo_controller" filename="libgazebo_ros_laser.so">
-        <topicName>/scan</topicName>
-        <frameName>hokuyo_link</frameName>
-      </plugin>
-    </sensor>
-  </gazebo>
-  <!-- -->
-  <joint name="camera_joint" type="fixed">
-    <origin xyz="0.1 0 0.2" rpy="0 0 0"/>
-    <parent link="chassis"/>
-    <child link="camera_link"/>
-  </joint>
-  <!-- Camera -->
-  <link name="camera_link">
-    <collision>
-      <origin xyz="0 0 0" rpy="0 0 0"/>
-      <geometry>
-    <box size="0.1 0.1 0.1"/>
-      </geometry>
-    </collision>
-    <visual>
-      <origin xyz="0 0 0" rpy="0 0 0"/>
-      <geometry>
-    <box size="0.1 0.1 0.1"/>
-      </geometry>
-      <material name="red"/>
-    </visual>
-    <inertial>
-      <mass value="1e-5" />
-      <origin xyz="0 0 0" rpy="0 0 0"/>
-      <inertia ixx="1e-6" ixy="0" ixz="0" iyy="1e-6" iyz="0" izz="1e-6" />
-    </inertial>
-  </link>
-   <xacro:property name="camera_link" value="0.05" /> <!-- Size of square 'camera' box -->
-  <!-- camera -->
-  <gazebo reference="camera_link">
-    <sensor type="camera" name="camera1">
-      <update_rate>30.0</update_rate>
-      <camera name="head">
-        <horizontal_fov>1.3962634</horizontal_fov>
-        <image>
-          <width>800</width>
-          <height>800</height>
-          <format>R8G8B8</format>
-        </image>
-        <clip>
-          <near>0.02</near>
-          <far>300</far>
-        </clip>
-        <noise>
-          <type>gaussian</type>
-          <!-- Noise is sampled independently per pixel on each frame.
+               <mean>0.0</mean>
+               <stddev>0.01</stddev>
+            </noise>
+         </ray>
+         <plugin name="gazebo_ros_head_hokuyo_controller" filename="libgazebo_ros_laser.so">
+            <topicName>/scan</topicName>
+            <frameName>hokuyo_link</frameName>
+         </plugin>
+      </sensor>
+   </gazebo>
+   <!-- joint Chassis-Camera -->
+   <joint name="camera_joint" type="fixed">
+      <origin xyz="0.22 0 0.1" rpy="0 0.3 0"/>
+      <parent link="chassis"/>
+      <child link="camera_link"/>
+   </joint>
+   <!-- Camera -->
+   <link name="camera_link">
+      <collision>
+         <origin xyz="0 0 0" rpy="0 0 0"/>
+         <geometry>
+            <box size="0.04 0.04 0.04"/>
+         </geometry>
+      </collision>
+      <visual>
+         <origin xyz="0 0 0" rpy="0 0 0"/>
+         <geometry>
+            <box size="0.04 0.04 0.04"/>
+         </geometry>
+         <material name="red"/>
+      </visual>
+      <inertial>
+         <mass value="1e-5" />
+         <origin xyz="0 0 0" rpy="0 0 0"/>
+         <inertia ixx="1e-6" ixy="0" ixz="0" iyy="1e-6" iyz="0" izz="1e-6" />
+      </inertial>
+   </link>
+   <xacro:property name="camera_link" value="0.4" /> <!-- Size of square 'camera' box -->
+   <!-- Plugin Camera -->
+   <gazebo reference="camera_link">
+      <sensor type="camera" name="camera1">
+         <update_rate>30.0</update_rate>
+         <camera name="head">
+            <horizontal_fov>1.3962634</horizontal_fov>
+            <image>
+               <width>800</width>
+               <height>800</height>
+               <format>R8G8B8</format>
+            </image>
+            <clip>
+               <near>0.02</near>
+               <far>300</far>
+            </clip>
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
Commit message: modif du lidar

File: workspaceRos/src/robot_description/urdf/robot.urdf (robot description, URDF)
Before this commit: robot monRobot, 8 links, 7 joints
Joints:
- joint hokuyo_joint: origin xyz=0 0 0.2 rpy=0 0 0 -> xyz=0 0 0.25 rpy=0 0 0

Commit message: ajout rapport_seance4 et modif position hokuyo

File: workspaceRos/src/robot_description/urdf/robot.urdf (robot description, URDF)
Before this commit: robot monRobot, 13 links, 12 joints
Links:
- added link hokuyo_support, mass 1e-5; collision cylinder length=0.05 radius=0.05; visual cylinder length=0.05 radius=0.05
- link hokuyo_link: geometry collision cylinder length=0.035 radius=0.05; visual cylinder length=0.035 radius=0.05
Joints:
- added joint support_hokuyo_joint: type fixed, parent chassis, child hokuyo_support, origin xyz=0 0 0.20 rpy=0 0 0, axis 0 1 -0.04
- joint cameraBras_joint: origin xyz=0 0 0.1 rpy=0 0 0 -> xyz=0 0 0.1 rpy=0 -1.7 0
- joint hokuyo_joint: origin xyz=0 0 0.22 rpy=0 0 0 -> xyz=0 0 0.041 rpy=0 0 0; parent chassis -> hokuyo_support
- joint joint_12: limit (none) -> lower=-3 upper=3.2 effort=5.0 velocity=1; type continuous -> revolute
- joint joint_23: limit lower=-0.2 upper=0.0 effort=10.0 velocity=0.5 -> lower=-1.0 upper=1.0 effort=10.0 velocity=0.5

File: workspaceRos/src/robot_description/urdf/robot.urdf.xacro (robot description, xacro)
@@ -135,6 +135,6 @@
    <!-- Joint Chassis-Support Hokuyo-->
    <joint name="support_hokuyo_joint" type="fixed">
-      <axis xyz="0 1 0" />
-      <origin xyz="0 0 0.22" rpy="0 0 0"/>
+      <axis xyz="0 1 -0.04" />
+      <origin xyz="0 0 0.20" rpy="0 0 0"/>
       <parent link="chassis"/>
       <child link="hokuyo_support"/>
@@ -145,5 +145,5 @@
          <origin xyz="0 0 -0.03" rpy="0 0 0"/>
          <geometry>
-    	    <cylinder radius="0.05" length="0.14"/>
+    	    <cylinder radius="0.05" length="0.05"/>
          </geometry>
       </collision>
@@ -151,5 +151,5 @@
          <origin xyz="0 0 -0.03" rpy="0 0 0"/>
          <geometry>
-            <cylinder radius="0.05" length="0.14"/>
+            <cylinder radius="0.05" length="0.05"/>
          </geometry>
       </visual>
@@ -163,5 +163,5 @@
    <joint name="hokuyo_joint" type="fixed">
       <axis xyz="0 1 0" />
-      <origin xyz="0 0 0.22" rpy="0 0 0"/>
+      <origin xyz="0 0 0.041" rpy="0 0 0"/>
       <parent link="hokuyo_support"/>
       <child link="hokuyo_link"/>
@@ -172,5 +172,5 @@
          <origin xyz="0 0 -0.03" rpy="0 0 0"/>
          <geometry>
-    	    <cylinder radius="0.05" length="0.05"/>
+    	    <cylinder radius="0.05" length="0.033"/>
          </geometry>
       </collision>
@@ -178,5 +178,5 @@
          <origin xyz="0 0 -0.03" rpy="0 0 0"/>
          <geometry>
-            <cylinder radius="0.05" length="0.05"/>
+            <cylinder radius="0.05" length="0.035"/>
          </geometry>
       </visual>
