Commit message: "bras contoller"

File: workspaceRos/src/robot_description/urdf/arm.xacro (robot description, xacro)
@@ -104,10 +104,10 @@
     </visual>
   </gazebo>
-  <joint name="joint_34" type="fixed">
+<joint name="joint_34" type="fixed">
     <origin xyz="0 0 ${length_3}" rpy="0 1.5707 0"/>
     <child link="laser"/>
     <parent link="arm_3_link"/>
   </joint>
-   <!--4th Link LASER-->
+    <!-- 4th Link LASER-->
   <link name="laser">
     <collision>
@@ -128,4 +128,30 @@
       <inertia ixx="1e-6" ixy="0" ixz="0" iyy="1e-6" iyz="0" izz="1e-6"/>
     </inertial>
-</link>
+  </link>
+  <!-- Controllers -->
+<gazebo>
+  <plugin name="gazebo_ros_control" filename="libgazebo_ros_control.so">
+    <robotNamespace>/my_robot</robotNamespace>
+  </plugin>
+</gazebo>
+  <transmission name="tran1">
+    <type>transmission_interface/SimpleTransmission</type>
+    <joint name="joint_12">
+      <hardwareInterface>hardware_interface/EffortJointInterface</hardwareInterface>
+    </joint>
+    <actuator name="motor1">
+      <hardwareInterface>hardware_interface/EffortJointInterface</hardwareInterface>
+      <mechanicalReduction>1</mechanicalReduction>
+    </actuator>
+  </transmission>
+  <transmission name="tran2">
+    <type>transmission_interface/SimpleTransmission</type>
+    <joint name="joint_23">
+      <hardwareInterface>hardware_interface/EffortJointInterface</hardwareInterface>
+    </joint>
+    <actuator name="motor2">
+      <hardwareInterface>hardware_interface/EffortJointInterface</hardwareInterface>
+      <mechanicalReduction>1</mechanicalReduction>
+    </actuator>
+</transmission>
 </robot>

File: workspaceRos/src/robot_description/urdf/robot.urdf.xacro (robot description, xacro)
@@ -277,4 +277,9 @@
    </gazebo>
   <!-- Controllers -->
+<gazebo>
+  <plugin name="gazebo_ros_control" filename="libgazebo_ros_control.so">
+    <robotNamespace>/my_robot</robotNamespace>
+  </plugin>
+</gazebo>
    <gazebo>
       <plugin name="wheels_controller" filename="libgazebo_ros_diff_drive.so">

Commit message: "controller issues"

File: workspaceRos/src/robot_description/urdf/arm.xacro (robot description, xacro)
@@ -74,5 +74,5 @@
     <origin xyz="0 0 ${length_2}" rpy="0 0 0"/>
     <axis xyz="0 0 1"/>
-    <limit effort="1000.0" lower="-0.2" upper="0.0" velocity="0.5"/>
+    <limit effort="1000.0" lower="-0.2" upper="1.0" velocity="0.5"/>
   </joint>
    <!--Third Link Verin entre 2 et 3-->
@@ -97,4 +97,5 @@
 </link>
   <gazebo reference="arm_3_link">
+    <!--<selfCollide>false</selfCollide> -->
     <visual>
       <material>
@@ -130,9 +131,9 @@
   </link>
   <!-- Controllers -->
-<gazebo>
-  <plugin name="gazebo_ros_control" filename="libgazebo_ros_control.so">
-    <robotNamespace>/rrbot</robotNamespace>
-  </plugin>
-</gazebo>
+  <gazebo>
+    <plugin name="gazebo_ros_control" filename="libgazebo_ros_control.so">
+      <robotNamespace>/rrbot</robotNamespace>
+    </plugin>
+  </gazebo>
   <transmission name="tran1">
     <type>transmission_interface/SimpleTransmission</type>

Commit message: last maj

File: workspaceRos/src/robot_description/urdf/arm.xacro (robot description, xacro)
@@ -4,5 +4,5 @@
   <!-- Constants for robot dimensions -->
   <xacro:property name="PI" value="3.1415926535897931"/>
-  <xacro:property name="mass_first_part" value="1" /> <!-- arbitrary value for mass -->
+  <xacro:property name="mass_first_part" value="0.01" /> <!-- arbitrary value for mass -->
   <xacro:property name="length_1" value="0.1" /> <!-- first arm -->
   <xacro:property name="length_2" value="0.15" /> <!-- second arm -->
@@ -35,7 +35,7 @@
     </visual>
     <inertial>
-      <mass value="1e-5"/>
+      <mass value="0.01"/>
       <origin rpy="0 0 0" xyz="0 0 0"/>
-      <inertia ixx="1e-6" ixy="0" ixz="0" iyy="1e-6" iyz="0" izz="1e-6"/>
+      <inertia ixx="0.001" ixy="0" ixz="0" iyy="0.001" iyz="0" izz="0.001"/>
     </inertial>
   </link>
@@ -50,10 +50,4 @@
  <!--second Link -->
   <link name="arm_2_link">
-    <collision>
-      <origin xyz="0 0 ${length_2 / 2}" rpy="0 0 0"/>
-      <geometry>
-        <cylinder length="${length_2}" radius="${radius}"/>
-      </geometry>
-    </collision>
     <visual>
       <origin xyz="0 0 ${length_2 / 2}" rpy="0 0 0"/>
@@ -64,7 +58,7 @@
     </visual>
     <inertial>
-      <mass value="1e-5"/>
+      <mass value="0.01"/>
       <origin rpy="0 0 0" xyz="0 0 0"/>
-      <inertia ixx="1e-6" ixy="0" ixz="0" iyy="1e-6" iyz="0" izz="1e-6"/>
+      <inertia ixx="0.001" ixy="0.001" ixz="0.001" iyy="0.001" iyz="0.001" izz="0.001"/>
     </inertial>
   </link>
@@ -74,14 +68,8 @@
     <origin xyz="0 0 ${length_2}" rpy="0 0 0"/>
     <axis xyz="0 0 1"/>
-    <limit effort="1000.0" lower="-0.2" upper="1.0" velocity="0.5"/>
+    <limit effort="10.0" lower="-0.2" upper="0.0" velocity="0.5"/>
   </joint>
    <!--Third Link Verin entre 2 et 3-->
   <link name="arm_3_link">
-    <collision>
-      <origin xyz="0 0 ${length_3 / 2}" rpy="0 0 0"/>
-      <geometry>
-        <cylinder length="${length_3}" radius="${radius}"/>
-      </geometry>
-    </collision>
     <visual>
       <origin xyz="0 0 ${length_3 / 2}" rpy="0 0 0"/>
@@ -91,7 +79,7 @@
     </visual>
     <inertial>
-      <mass value="1e-5"/>
+      <mass value="0.01"/>
       <origin rpy="0 0 0" xyz="0 0 0"/>
-      <inertia ixx="1e-6" ixy="0" ixz="0" iyy="1e-6" iyz="0" izz="1e-6"/>
+      <inertia ixx="0.001" ixy="0.001" ixz="0.001" iyy="0.001" iyz="0.001" izz="0.001"/>
     </inertial>
 </link>
@@ -125,7 +113,7 @@
     </visual>
     <inertial>
-      <mass value="1e-5"/>
+      <mass value="0.01"/>
       <origin rpy="0 0 0" xyz="0 0 0"/>
-      <inertia ixx="1e-6" ixy="0" ixz="0" iyy="1e-6" iyz="0" izz="1e-6"/>
+      <inertia ixx="0.001" ixy="0.001" ixz="0.001" iyy="0.001" iyz="0.001" izz="0.001"/>
     </inertial>
   </link>

File: workspaceRos/src/robot_description/urdf/robot.urdf.xacro (robot description, xacro)
@@ -30,5 +30,5 @@
          </geometry>
       </visual>
-     <xacro:default_inertial mass="2.0"/>
+     <xacro:default_inertial mass="10.0"/>
    </link>
    <!-- Roue Libre-->

Commit message: "controller pid"

File: workspaceRos/src/robot_description/urdf/arm.xacro (robot description, xacro)
@@ -16,5 +16,5 @@
     <inertial>
       <mass value="${mass}" />
-      <inertia ixx="0.01" ixy="0.0" ixz="0.0" iyy="0.01" iyz="0.0" izz="0.01" />
+      <inertia ixx="0.01" ixy="0.0001" ixz="0.0001" iyy="0.01" iyz="0.0001" izz="0.01" />
     </inertial>
   </xacro:macro>
@@ -41,9 +41,10 @@
   </link>
   <!--xacro:property name="arm_1_link" value="0.05" /--> <!-- Size of square 'camera' box -->
-  <joint name="joint_12" type="continuous">
+  <joint name="joint_12" type="revolute">
     <parent link="arm_1_link"/>
     <child link="arm_2_link"/>
     <origin xyz="0 0 ${length_1/2}" rpy="0 1.5707 0"/>
     <axis xyz="1 0 0"/>
+    <limit effort="5.0" lower="-3" upper="3.2" velocity="1"/>
     <!--dynamics damping="0.7"/-->
   </joint>

File: workspaceRos/src/robot_description/urdf/robot.urdf.xacro (robot description, xacro)
@@ -6,5 +6,5 @@
     <inertial>
       <mass value="${mass}" />
-      <inertia ixx="0.01" ixy="0.0" ixz="0.0" iyy="0.01" iyz="0.0" izz="0.01" />
+      <inertia ixx="0.01" ixy="0.0001" ixz="0.0001" iyy="0.01" iyz="0.0001" izz="0.01" />
     </inertial>
   </xacro:macro>

Commit message: "reglage positionnement bras"

File: workspaceRos/src/robot_description/urdf/arm.xacro (robot description, xacro)
@@ -69,5 +69,5 @@
     <origin xyz="0 0 ${length_2}" rpy="0 0 0"/>
     <axis xyz="0 0 1"/>
-    <limit effort="10.0" lower="-0.2" upper="0.0" velocity="0.5"/>
+    <limit effort="10.0" lower="-1.0" upper="1.0" velocity="0.5"/>
   </joint>
    <!--Third Link Verin entre 2 et 3-->

Commit message: position initial du bras repliée

File: workspaceRos/src/robot_description/urdf/arm.xacro (robot description, xacro)
@@ -6,5 +6,5 @@
   <xacro:property name="mass_first_part" value="0.01" /> <!-- arbitrary value for mass -->
   <xacro:property name="length_1" value="0.1" /> <!-- first arm -->
-  <xacro:property name="length_2" value="0.15" /> <!-- second arm -->
+  <xacro:property name="length_2" value="0.20" /> <!-- second arm -->
   <xacro:property name="length_3" value="0.25" /> <!-- third arm -->
   <xacro:property name="length_4" value="0.1" /> <!-- laser arm -->
@@ -44,5 +44,5 @@
     <parent link="arm_1_link"/>
     <child link="arm_2_link"/>
-    <origin xyz="0 0 ${length_1/2}" rpy="0 1.5707 0"/>
+    <origin xyz="0 0 ${length_1/2}" rpy="0 1.5707 3.1415"/>
     <axis xyz="1 0 0"/>
     <limit effort="5.0" lower="-3" upper="3.2" velocity="1"/>

Commit message: dernière version dev testée

File: workspaceRos/src/robot_description/urdf/arm.xacro (robot description, xacro)
@@ -10,5 +10,6 @@
   <xacro:property name="length_4" value="0.1" /> <!-- laser arm -->
   <xacro:property name="arm_position" value="0.17" /> <!-- first arm -->
-  <xacro:property name="radius" value="0.02" /> <!-- Link 3 -->
+  <xacro:property name="radius" value="0.02" />
+  <xacro:property name="radius_arm_3" value="0.018" />
   <xacro:property name="camera_link" value="0.05" /> <!-- Size of square 'camera' box -->
   <xacro:property name="axel_offset" value="0.05" /> <!-- Space btw top of beam and the each joint -->
@@ -76,5 +77,5 @@
       <origin xyz="0 0 ${length_3 / 2}" rpy="0 0 0"/>
       <geometry>
-        <cylinder length="${length_3}" radius="${radius}"/>
+        <cylinder length="${length_3}" radius="${radius_arm_3}"/>
       </geometry>
     </visual>
